Commit message: fix(description): Add better model for simulation
Use URDF, for stl

File: src/amphi_description/urdf/amphi.urdf (robot description, URDF)
Before this commit: robot amphibious_screw_robot, 3 links, 2 joints
Links:
- removed link base_link
- removed link left_screw
- removed link right_screw
- added link Amphi_body, mass 7.212459883295273; collision mesh filename=package://amphi_description/urdf/meshes/Amphi_body-v14.stl scale=0.001 0.001 0.001; visual mesh filename=package://amphi_description/urdf/meshes/Amphi_body-v14.stl scale=0.001 0.001 0.001
- added link left-back-support, mass 0.23800029540907736; collision mesh filename=package://amphi_description/urdf/meshes/left-back-support-v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 scale=0.001 0.001 0.001; visual mesh filename=package://amphi_description/urdf/meshes/left-back-support-v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 scale=0.001 0.001 0.001
- added link left-front-support, mass 0.1258063436309947; collision mesh filename=package://amphi_description/urdf/meshes/left-front-support-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 scale=0.001 0.001 0.001; visual mesh filename=package://amphi_description/urdf/meshes/left-front-support-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 scale=0.001 0.001 0.001
- added link left-wheel, mass 5.030310348521676; collision mesh filename=package://amphi_description/urdf/meshes/left-wheel-v4.stl scale=0.001 0.001 0.001; visual mesh filename=package://amphi_description/urdf/meshes/left-wheel-v4.stl scale=0.001 0.001 0.001
- added link right-back-support, mass 0.23800029540906284; collision mesh filename=package://amphi_description/urdf/meshes/right--back-support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 scale=0.001 0.001 0.001; visual mesh filename=package://amphi_description/urdf/meshes/right--back-support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 scale=0.001 0.001 0.001
- added link right-front-support, mass 0.12580634363099644; collision mesh filename=package://amphi_description/urdf/meshes/right-front-support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 scale=0.001 0.001 0.001; visual mesh filename=package://amphi_description/urdf/meshes/right-front-support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 scale=0.001 0.001 0.001
- added link right-wheel, mass 5.029486679133445; collision mesh filename=package://amphi_description/urdf/meshes/right-wheel-v5.stl scale=0.001 0.001 0.001; visual mesh filename=package://amphi_description/urdf/meshes/right-wheel-v5.stl scale=0.001 0.001 0.001
- added link shaft-left, mass 0.02841005068494322; collision mesh filename=package://amphi_description/urdf/meshes/shaft-v4.stl scale=0.001 0.001 0.001; visual mesh filename=package://amphi_description/urdf/meshes/shaft-v4.stl scale=0.001 0.001 0.001
- added link shaft-right, mass 0.02841005068494322; collision mesh filename=package://amphi_description/urdf/meshes/shaft-v4.stl scale=0.001 0.001 0.001; visual mesh filename=package://amphi_description/urdf/meshes/shaft-v4.stl scale=0.001 0.001 0.001
Joints:
- removed joint left_screw_joint
- removed joint right_screw_joint
- added joint left-front-support-joint: type fixed, parent Amphi_body, child left-front-support, origin xyz=-0.23 -0.009 -0.016 rpy=3.14 0.0 3.14
- added joint left-wheel-joint: type continuous, parent shaft-left, child left-wheel, origin xyz=0.0 0.013 0.0 rpy=1.57 0.0 0.0, axis 0 0  1
- added joint right-front-support-joint: type fixed, parent Amphi_body, child right-front-support, origin xyz=-0.040 -0.029 -0.015 rpy=0.0 3.14 0.0
- added joint right-wheel-joint: type continuous, parent shaft-right, child right-wheel, origin xyz=0.0 0.013 0.0 rpy=1.57 0.0 0.0, axis 0 0  1
- added joint shaft-left-back-joint: type fixed, parent shaft-left, child left-back-support, origin xyz=0.06 -0.23 -0.11 rpy=0.0 0.0 0.0
- added joint shaft-left-joint: type fixed, parent left-front-support, child shaft-left, origin xyz=0.1 0.01 0.07 rpy=0.0 0.0 3.14
- added joint shaft-right-back-joint: type fixed, parent shaft-right, child right-back-support, origin xyz=-0.1 -0.21 -0.11 rpy=0.0 0.0 0.0
- added joint shaft-right-joint: type fixed, parent right-front-support, child shaft-right, origin xyz=-0.059 0.03 0.0715 rpy=0.0 0.0 3.14
